Commit message: floating 追加

File: xacro/KHR3_001.xacro (robot description, xacro)
@@ -4,4 +4,6 @@
 <xacro:include filename="$(find KHR3_001_description)/xacro/KHR3_001.trans" />
 <xacro:include filename="$(find KHR3_001_description)/xacro/KHR3_001.gazebo" />
+ <!-- Description of robot -->
+<link name="base_footprint"/>
 <link name="base_link">
   <inertial>
@@ -504,4 +506,9 @@
   </collision>
 </link>
+<joint name="base_joint0" type="floating">
+        <parent link="base_footprint"/>
+        <child link="base_link"/>
+        <origin rpy="0 0 0" xyz="0 0 0"/>
+  </joint>
 <joint name="base_link1" type="continuous">
   <origin xyz="0.010956 0.009542 0.29475" rpy="0 0 0"/>

Commit message: meridian-ROS サンプル動作確認

File: xacro/KHR3_001.xacro (robot description, xacro)
@@ -511,5 +511,5 @@
         <origin rpy="0 0 0" xyz="0 0 0"/>
   </joint>
-<joint name="base_link1" type="continuous">
+<joint name="c_chest_yaw" type="continuous">
   <origin xyz="0.010956 0.009542 0.29475" rpy="0 0 0"/>
   <parent link="base_link"/>
@@ -533,5 +533,5 @@
   <axis xyz="0.0 -0.0 1.0"/>
 </joint>
-<joint name="l_shouluder_pitch" type="continuous">
+<joint name="l_shoulder_pitch" type="continuous">
   <origin xyz="0.0115 0.0489 0.04775" rpy="0 0 0"/>
   <parent link="c_chest_c_1"/>
@@ -539,5 +539,5 @@
   <axis xyz="-0.0 1.0 0.0"/>
 </joint>
-<joint name="l_shouluder_roll" type="continuous">
+<joint name="l_shoulder_roll" type="continuous">
   <origin xyz="0.01575 0.025 0.0" rpy="0 0 0"/>
   <parent link="l_shoulder_v5_1"/>
@@ -557,5 +557,5 @@
   <axis xyz="-0.0 1.0 0.0"/>
 </joint>
-<joint name="r_shouluder_pitch" type="continuous">
+<joint name="r_shoulder_pitch" type="continuous">
   <origin xyz="0.0115 -0.0489 0.04775" rpy="0 0 0"/>
   <parent link="c_chest_c_1"/>
@@ -563,5 +563,5 @@
   <axis xyz="0.0 -1.0 -0.0"/>
 </joint>
-<joint name="r_shouluder_roll" type="continuous">
+<joint name="r_shoulder_roll" type="continuous">
   <origin xyz="0.01575 -0.025 0.0" rpy="0 0 0"/>
   <parent link="r_shoulder_v4_1"/>
