Commit message: 論文 直前

File: xacro/khr3_001 (コピー).xacro (robot description, xacro)
@@ -1,7 +1,7 @@
 <?xml version="1.0" ?>
-<robot name="KHR3_001" xmlns:xacro="http://www.ros.org/wiki/xacro">
-<xacro:include filename="$(find KHR3_001_description)/xacro/materials.xacro" />
-<xacro:include filename="$(find KHR3_001_description)/xacro/KHR3_001.trans" />
-<xacro:include filename="$(find KHR3_001_description)/xacro/KHR3_001.gazebo" />
+<robot name="khr3_001" xmlns:xacro="http://www.ros.org/wiki/xacro">
+<xacro:include filename="$(find choreonoid_ros_khr3)/xacro/materials.xacro" />
+<xacro:include filename="$(find choreonoid_ros_khr3)/xacro/khr3_001.trans" />
+<xacro:include filename="$(find choreonoid_ros_khr3)/xacro/khr3_001.gazebo" />
  <!-- Description of robot -->
 <link name="base_footprint"/>
@@ -15,16 +15,16 @@
     <origin xyz="0 0 0" rpy="0 0 0"/>
     <geometry>
-      <mesh filename="package://KHR3_001_description/meshes/base_link.stl" scale="0.001 0.001 0.001"/>
-    </geometry>
-    <material name="silver"/>
+      <mesh filename="package://choreonoid_ros_khr3/meshes/base_link.stl" scale="0.001 0.001 0.001"/>
+    </geometry>
+    <material name="black"/>
   </visual>
   <collision>
     <origin xyz="0 0 0" rpy="0 0 0"/>
     <geometry>
-      <mesh filename="package://KHR3_001_description/meshes/base_link.stl" scale="0.001 0.001 0.001"/>
-    </geometry>
-  </collision>
-</link>
-<link name="c_chest_c_1">
+      <mesh filename="package://choreonoid_ros_khr3/meshes/base_link.stl" scale="0.001 0.001 0.001"/>
+    </geometry>
+  </collision>
+</link>
+<link name="c_chest_c">
   <inertial>
     <origin xyz="-9.07564737343998e-05 -4.299695898109246e-08 0.04371354326547944" rpy="0 0 0"/>
@@ -35,5 +35,5 @@
     <origin xyz="-0.010956 -0.009542 -0.29475" rpy="0 0 0"/>
     <geometry>
-      <mesh filename="package://KHR3_001_description/meshes/c_chest_c_1.stl" scale="0.001 0.001 0.001"/>
+      <mesh filename="package://choreonoid_ros_khr3/meshes/c_chest_c_1.stl" scale="0.001 0.001 0.001"/>
     </geometry>
     <material name="silver"/>
@@ -42,9 +42,9 @@
     <origin xyz="-0.010956 -0.009542 -0.29475" rpy="0 0 0"/>
     <geometry>
-      <mesh filename="package://KHR3_001_description/meshes/c_chest_c_1.stl" scale="0.001 0.001 0.001"/>
-    </geometry>
-  </collision>
-</link>
-<link name="c_chest_b_1">
+      <mesh filename="package://choreonoid_ros_khr3/meshes/c_chest_c_1.stl" scale="0.001 0.001 0.001"/>
+    </geometry>
+  </collision>
+</link>
+<link name="c_chest_b">
   <inertial>
     <origin xyz="-0.027362562372520854 2.840518613928325e-06 0.004477857770456339" rpy="0 0 0"/>
@@ -55,16 +55,16 @@
     <origin xyz="0.015044 -0.009542 -0.326" rpy="0 0 0"/>
     <geometry>
-      <mesh filename="package://KHR3_001_description/meshes/c_chest_b_1.stl" scale="0.001 0.001 0.001"/>
-    </geometry>
-    <material name="silver"/>
+      <mesh filename="package://choreonoid_ros_khr3/meshes/c_chest_b_1.stl" scale="0.001 0.001 0.001"/>
+    </geometry>
+    <material name="black"/>
   </visual>
   <collision>
     <origin xyz="0.015044 -0.009542 -0.326" rpy="0 0 0"/>
     <geometry>
-      <mesh filename="package://KHR3_001_description/meshes/c_chest_b_1.stl" scale="0.001 0.001 0.001"/>
-    </geometry>
-  </collision>
-</link>
-<link name="c_chest_a_1">
+      <mesh filename="package://choreonoid_ros_khr3/meshes/c_chest_b_1.stl" scale="0.001 0.001 0.001"/>
+    </geometry>
+  </collision>
+</link>
+<link name="c_chest_a">
   <inertial>
     <origin xyz="0.004546800382866728 -4.1161282904669805e-08 -0.0024788373011201403" rpy="0 0 0"/>
@@ -75,5 +75,5 @@
     <origin xyz="-0.036956 -0.009542 -0.326" rpy="0 0 0"/>
     <geometry>
-      <mesh filename="package://KHR3_001_description/meshes/c_chest_a_1.stl" scale="0.001 0.001 0.001"/>
+      <mesh filename="package://choreonoid_ros_khr3/meshes/c_chest_a_1.stl" scale="0.001 0.001 0.001"/>
     </geometry>
     <material name="silver"/>
@@ -82,9 +82,9 @@
     <origin xyz="-0.036956 -0.009542 -0.326" rpy="0 0 0"/>
     <geometry>
-      <mesh filename="package://KHR3_001_description/meshes/c_chest_a_1.stl" scale="0.001 0.001 0.001"/>
-    </geometry>
-  </collision>
-</link>
-<link name="c_head_a_1">
+      <mesh filename="package://choreonoid_ros_khr3/meshes/c_chest_a_1.stl" scale="0.001 0.001 0.001"/>
+    </geometry>
+  </collision>
+</link>
+<link name="c_head_a">
   <inertial>
     <origin xyz="0.003079433021973575 -4.3073247395913894e-08 0.022888877386975093" rpy="0 0 0"/>
@@ -95,5 +95,5 @@
     <origin xyz="-0.022456 -0.009542 -0.35425" rpy="0 0 0"/>
     <geometry>
-      <mesh filename="package://KHR3_001_description/meshes/c_head_a_1.stl" scale="0.001 0.001 0.001"/>
+      <mesh filename="package://choreonoid_ros_khr3/meshes/c_head_a_1.stl" scale="0.001 0.001 0.001"/>
     </geometry>
     <material name="silver"/>
@@ -102,9 +102,9 @@
     <origin xyz="-0.022456 -0.009542 -0.35425" rpy="0 0 0"/>
     <geometry>
-      <mesh filename="package://KHR3_001_description/meshes/c_head_a_1.stl" scale="0.001 0.001 0.001"/>
-    </geometry>
-  </collision>
-</link>
-<link name="l_shoulder_v5_1">
+      <mesh filename="package://choreonoid_ros_khr3/meshes/c_head_a_1.stl" scale="0.001 0.001 0.001"/>
+    </geometry>
+  </collision>
+</link>
+<link name="l_shoulder">
   <inertial>
     <origin xyz="0.00016940373751364937 0.008747288709026461 3.2529534621517087e-14" rpy="0 0 0"/>
@@ -115,16 +115,16 @@
     <origin xyz="-0.022456 -0.058442 -0.3425" rpy="0 0 0"/>
     <geometry>
-      <mesh filename="package://KHR3_001_description/meshes/l_shoulder_v5_1.stl" scale="0.001 0.001 0.001"/>
-    </geometry>
-    <material name="silver"/>
+      <mesh filename="package://choreonoid_ros_khr3/meshes/l_shoulder_v5_1.stl" scale="0.001 0.001 0.001"/>
+    </geometry>
+    <material name="black"/>
   </visual>
   <collision>
     <origin xyz="-0.022456 -0.058442 -0.3425" rpy="0 0 0"/>
     <geometry>
-      <mesh filename="package://KHR3_001_description/meshes/l_shoulder_v5_1.stl" scale="0.001 0.001 0.001"/>
-    </geometry>
-  </collision>
-</link>
-<link name="l_upperarm_v4_1">
+      <mesh filename="package://choreonoid_ros_khr3/meshes/l_shoulder_v5_1.stl" scale="0.001 0.001 0.001"/>
+    </geometry>
+  </collision>
+</link>
+<link name="l_upperarm">
   <inertial>
     <origin xyz="-0.02256531849252991 -4.2996961130414846e-08 -0.03564584515249991" rpy="0 0 0"/>
@@ -135,5 +135,5 @@
     <origin xyz="-0.038206 -0.083442 -0.3425" rpy="0 0 0"/>
     <geometry>
-      <mesh filename="package://KHR3_001_description/meshes/l_upperarm_v4_1.stl" scale="0.001 0.001 0.001"/>
+      <mesh filename="package://choreonoid_ros_khr3/meshes/l_upperarm_v4_1.stl" scale="0.001 0.001 0.001"/>
     </geometry>
     <material name="silver"/>
@@ -142,9 +142,9 @@
     <origin xyz="-0.038206 -0.083442 -0.3425" rpy="0 0 0"/>
     <geometry>
-      <mesh filename="package://KHR3_001_description/meshes/l_upperarm_v4_1.stl" scale="0.001 0.001 0.001"/>
-    </geometry>
-  </collision>
-</link>
-<link name="l_elbow_v4_1">
+      <mesh filename="package://choreonoid_ros_khr3/meshes/l_upperarm_v4_1.stl" scale="0.001 0.001 0.001"/>
+    </geometry>
+  </collision>
+</link>
+<link name="l_elbow">
   <inertial>
     <origin xyz="5.745484729775818e-05 -4.299695875731313e-08 -0.012574921301198305" rpy="0 0 0"/>
@@ -155,16 +155,16 @@
     <origin xyz="-0.022206 -0.083442 -0.27075" rpy="0 0 0"/>
     <geometry>
-      <mesh filename="package://KHR3_001_description/meshes/l_elbow_v4_1.stl" scale="0.001 0.001 0.001"/>
-    </geometry>
-    <material name="silver"/>
+      <mesh filename="package://choreonoid_ros_khr3/meshes/l_elbow_v4_1.stl" scale="0.001 0.001 0.001"/>
+    </geometry>
+    <material name="black"/>
   </visual>
   <collision>
     <origin xyz="-0.022206 -0.083442 -0.27075" rpy="0 0 0"/>
     <geometry>
-      <mesh filename="package://KHR3_001_description/meshes/l_elbow_v4_1.stl" scale="0.001 0.001 0.001"/>
-    </geometry>
-  </collision>
-</link>
-<link name="l_lowerarm_v7_1">
+      <mesh filename="package://choreonoid_ros_khr3/meshes/l_elbow_v4_1.stl" scale="0.001 0.001 0.001"/>
+    </geometry>
+  </collision>
+</link>
+<link name="l_lowerarm">
   <inertial>
     <origin xyz="0.00017641899363149416 -0.0156924274010031 -0.04569649848488025" rpy="0 0 0"/>
@@ -175,5 +175,5 @@
     <origin xyz="-0.033706 -0.099692 -0.25625" rpy="0 0 0"/>
     <geometry>
-      <mesh filename="package://KHR3_001_description/meshes/l_lowerarm_v7_1.stl" scale="0.001 0.001 0.001"/>
+      <mesh filename="package://choreonoid_ros_khr3/meshes/l_lowerarm_v7_1.stl" scale="0.001 0.001 0.001"/>
     </geometry>
     <material name="silver"/>
@@ -182,9 +182,9 @@
     <origin xyz="-0.033706 -0.099692 -0.25625" rpy="0 0 0"/>
     <geometry>
-      <mesh filename="package://KHR3_001_description/meshes/l_lowerarm_v7_1.stl" scale="0.001 0.001 0.001"/>
-    </geometry>
-  </collision>
-</link>
-<link name="r_shoulder_v4_1">
+      <mesh filename="package://choreonoid_ros_khr3/meshes/l_lowerarm_v7_1.stl" scale="0.001 0.001 0.001"/>
+    </geometry>
+  </collision>
+</link>
+<link name="r_shoulder">
   <inertial>
     <origin xyz="0.00016940373733528857 -0.008747374702943796 5.306866057708248e-14" rpy="0 0 0"/>
@@ -195,16 +195,16 @@
     <origin xyz="-0.022456 0.039358 -0.3425" rpy="0 0 0"/>
     <geometry>
-      <mesh filename="package://KHR3_001_description/meshes/r_shoulder_v4_1.stl" scale="0.001 0.001 0.001"/>
-    </geometry>
-    <material name="silver"/>
+      <mesh filename="package://choreonoid_ros_khr3/meshes/r_shoulder_v4_1.stl" scale="0.001 0.001 0.001"/>
+    </geometry>
+    <material name="black"/>
   </visual>
   <collision>
     <origin xyz="-0.022456 0.039358 -0.3425" rpy="0 0 0"/>
     <geometry>
-      <mesh filename="package://KHR3_001_description/meshes/r_shoulder_v4_1.stl" scale="0.001 0.001 0.001"/>
-    </geometry>
-  </collision>
-</link>
-<link name="r_upperarm_v3_1">
+      <mesh filename="package://choreonoid_ros_khr3/meshes/r_shoulder_v4_1.stl" scale="0.001 0.001 0.001"/>
+    </geometry>
+  </collision>
+</link>
+<link name="r_upperarm">
   <inertial>
     <origin xyz="-0.022565318492529688 -4.2996961074903695e-08 -0.03564584515249991" rpy="0 0 0"/>
@@ -215,5 +215,5 @@
     <origin xyz="-0.038206 0.064358 -0.3425" rpy="0 0 0"/>
     <geometry>
-      <mesh filename="package://KHR3_001_description/meshes/r_upperarm_v3_1.stl" scale="0.001 0.001 0.001"/>
+      <mesh filename="package://choreonoid_ros_khr3/meshes/r_upperarm_v3_1.stl" scale="0.001 0.001 0.001"/>
     </geometry>
     <material name="silver"/>
@@ -222,9 +222,9 @@
     <origin xyz="-0.038206 0.064358 -0.3425" rpy="0 0 0"/>
     <geometry>
-      <mesh filename="package://KHR3_001_description/meshes/r_upperarm_v3_1.stl" scale="0.001 0.001 0.001"/>
-    </geometry>
-  </collision>
-</link>
-<link name="r_elbow_v4_1">
+      <mesh filename="package://choreonoid_ros_khr3/meshes/r_upperarm_v3_1.stl" scale="0.001 0.001 0.001"/>
+    </geometry>
+  </collision>
+</link>
+<link name="r_elbow">
   <inertial>
     <origin xyz="5.7454847330103836e-05 -4.2996958674046404e-08 -0.012574921301198305" rpy="0 0 0"/>
@@ -235,16 +235,16 @@
     <origin xyz="-0.022206 0.064358 -0.27075" rpy="0 0 0"/>
     <geometry>
-      <mesh filename="package://KHR3_001_description/meshes/r_elbow_v4_1.stl" scale="0.001 0.001 0.001"/>
-    </geometry>
-    <material name="silver"/>
+      <mesh filename="package://choreonoid_ros_khr3/meshes/r_elbow_v4_1.stl" scale="0.001 0.001 0.001"/>
+    </geometry>
+    <material name="black"/>
   </visual>
   <collision>
     <origin xyz="-0.022206 0.064358 -0.27075" rpy="0 0 0"/>
     <geometry>
-      <mesh filename="package://KHR3_001_description/meshes/r_elbow_v4_1.stl" scale="0.001 0.001 0.001"/>
-    </geometry>
-  </collision>
-</link>
-<link name="r_lowerarm_v5_1">
+      <mesh filename="package://choreonoid_ros_khr3/meshes/r_elbow_v4_1.stl" scale="0.001 0.001 0.001"/>
+    </geometry>
+  </collision>
+</link>
+<link name="r_lowerarm">
   <inertial>
     <origin xyz="0.00017641899364317232 0.01569234140705124 -0.04569649848495705" rpy="0 0 0"/>
@@ -255,5 +255,5 @@
     <origin xyz="-0.033706 0.080608 -0.25625" rpy="0 0 0"/>
     <geometry>
-      <mesh filename="package://KHR3_001_description/meshes/r_lowerarm_v5_1.stl" scale="0.001 0.001 0.001"/>
+      <mesh filename="package://choreonoid_ros_khr3/meshes/r_lowerarm_v5_1.stl" scale="0.001 0.001 0.001"/>
     </geometry>
     <material name="silver"/>
@@ -262,9 +262,9 @@
     <origin xyz="-0.033706 0.080608 -0.25625" rpy="0 0 0"/>
     <geometry>
-      <mesh filename="package://KHR3_001_description/meshes/r_lowerarm_v5_1.stl" scale="0.001 0.001 0.001"/>
-    </geometry>
-  </collision>
-</link>
-<link name="l_hipjointupper_v4_1">
+      <mesh filename="package://choreonoid_ros_khr3/meshes/r_lowerarm_v5_1.stl" scale="0.001 0.001 0.001"/>
+    </geometry>
+  </collision>
+</link>
+<link name="l_hipjointupper">
   <inertial>
     <origin xyz="3.293764515496962e-05 -0.0011113374509284651 -0.007400199793976242" rpy="0 0 0"/>
@@ -275,5 +275,5 @@
     <origin xyz="-0.010956 -0.031242 -0.25575" rpy="0 0 0"/>
     <geometry>
-      <mesh filename="package://KHR3_001_description/meshes/l_hipjointupper_v4_1.stl" scale="0.001 0.001 0.001"/>
+      <mesh filename="package://choreonoid_ros_khr3/meshes/l_hipjointupper_v4_1.stl" scale="0.001 0.001 0.001"/>
     </geometry>
     <material name="silver"/>
@@ -282,9 +282,9 @@
     <origin xyz="-0.010956 -0.031242 -0.25575" rpy="0 0 0"/>
     <geometry>
-      <mesh filename="package://KHR3_001_description/meshes/l_hipjointupper_v4_1.stl" scale="0.001 0.001 0.001"/>
-    </geometry>
-  </collision>
-</link>
-<link name="l_hipjointlower_v4_1">
+      <mesh filename="package://choreonoid_ros_khr3/meshes/l_hipjointupper_v4_1.stl" scale="0.001 0.001 0.001"/>
+    </geometry>
+  </collision>
+</link>
+<link name="l_hipjointlower">
   <inertial>
     <origin xyz="-0.016250242301438553 0.011463181378816707 -0.0066539419866288585" rpy="0 0 0"/>
@@ -295,16 +295,16 @@
     <origin xyz="-0.027656 -0.027242 -0.233" rpy="0 0 0"/>
     <geometry>
-      <mesh filename="package://KHR3_001_description/meshes/l_hipjointlower_v4_1.stl" scale="0.001 0.001 0.001"/>
-    </geometry>
-    <material name="silver"/>
+      <mesh filename="package://choreonoid_ros_khr3/meshes/l_hipjointlower_v4_1.stl" scale="0.001 0.001 0.001"/>
+    </geometry>
+    <material name="black"/>
   </visual>
   <collision>
     <origin xyz="-0.027656 -0.027242 -0.233" rpy="0 0 0"/>
     <geometry>
-      <mesh filename="package://KHR3_001_description/meshes/l_hipjointlower_v4_1.stl" scale="0.001 0.001 0.001"/>
-    </geometry>
-  </collision>
-</link>
-<link name="l_upperreg_v3_1">
+      <mesh filename="package://choreonoid_ros_khr3/meshes/l_hipjointlower_v4_1.stl" scale="0.001 0.001 0.001"/>
+    </geometry>
+  </collision>
+</link>
+<link name="l_upperreg">
   <inertial>
     <origin xyz="0.002589780466551929 -0.016500042996958703 -0.03375567398425394" rpy="0 0 0"/>
@@ -315,5 +315,5 @@
     <origin xyz="-0.011406 -0.054742 -0.1935" rpy="0 0 0"/>
     <geometry>
-      <mesh filename="package://KHR3_001_description/meshes/l_upperreg_v3_1.stl" scale="0.001 0.001 0.001"/>
+      <mesh filename="package://choreonoid_ros_khr3/meshes/l_upperreg_v3_1.stl" scale="0.001 0.001 0.001"/>
     </geometry>
     <material name="silver"/>
@@ -322,9 +322,9 @@
     <origin xyz="-0.011406 -0.054742 -0.1935" rpy="0 0 0"/>
     <geometry>
-      <mesh filename="package://KHR3_001_description/meshes/l_upperreg_v3_1.stl" scale="0.001 0.001 0.001"/>
-    </geometry>
-  </collision>
-</link>
-<link name="l_lowerreg_v5_1">
+      <mesh filename="package://choreonoid_ros_khr3/meshes/l_upperreg_v3_1.stl" scale="0.001 0.001 0.001"/>
+    </geometry>
+  </collision>
+</link>
+<link name="l_lowerreg">
   <inertial>
     <origin xyz="0.0044805681524230055 -0.015970110512676966 -0.04182100713444817" rpy="0 0 0"/>
@@ -335,16 +335,16 @@
     <origin xyz="-0.011406 -0.054742 -0.1285" rpy="0 0 0"/>
     <geometry>
-      <mesh filename="package://KHR3_001_description/meshes/l_lowerreg_v5_1.stl" scale="0.001 0.001 0.001"/>
-    </geometry>
-    <material name="silver"/>
+      <mesh filename="package://choreonoid_ros_khr3/meshes/l_lowerreg_v5_1.stl" scale="0.001 0.001 0.001"/>
+    </geometry>
+    <material name="black"/>
   </visual>
   <collision>
     <origin xyz="-0.011406 -0.054742 -0.1285" rpy="0 0 0"/>
     <geometry>
-      <mesh filename="package://KHR3_001_description/meshes/l_lowerreg_v5_1.stl" scale="0.001 0.001 0.001"/>
-    </geometry>
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
File: xacro/materials.xacro (robot description, xacro)
@@ -1,6 +1,12 @@
 <?xml version="1.0" ?>
-<robot name="KHR3_001" xmlns:xacro="http://www.ros.org/wiki/xacro" >
+<robot name="khr3_001" xmlns:xacro="http://www.ros.org/wiki/xacro" >
 <material name="silver">
   <color rgba="0.700 0.700 0.700 1.000"/>
 </material>
+<material name="white">
+        <color rgba="1.0 1.0 1.0 1.0"/>
+    </material>
+<material name="black">
+        <color rgba="0.0 0.0 0.0 1.0"/>
+    </material>
 </robot>
