Commit message: 2022年度吉田修論最終

File: xacro/khr3_001.xacro (robot description, xacro)
@@ -566,5 +566,5 @@
   <parent link="base_link"/>
   <child link="l_hipjointupper"/>
-  <axis xyz="-0.0 0.0 -1.0"/>
+  <axis xyz="-0.0 0.0 1.0"/>
   <limit effort="1000" lower="${radians(-90)}" upper="${radians(90)}" velocity="100.0"/>
 </joint>
@@ -615,5 +615,5 @@
   <parent link="c_chest_c"/>
   <child link="r_shoulder"/>
-  <axis xyz="0.0 -1.0 -0.0"/>
+  <axis xyz="0.0 1.0 -0.0"/>
   <limit effort="1000" lower="${radians(-90)}" upper="${radians(90)}" velocity="100.0"/>
 </joint>
@@ -622,5 +622,5 @@
   <parent link="r_shoulder"/>
   <child link="r_upperarm"/>
-  <axis xyz="1.0 0.0 0.0"/>
+  <axis xyz="-1.0 0.0 0.0"/>
   <limit effort="1000" lower="${radians(-90)}" upper="${radians(90)}" velocity="100.0"/>
 </joint>
@@ -629,5 +629,5 @@
   <parent link="r_upperarm"/>
   <child link="r_elbow"/>
-  <axis xyz="-0.0 0.0 1.0"/>
+  <axis xyz="-0.0 0.0 -1.0"/>
   <limit effort="1000" lower="${radians(-90)}" upper="${radians(90)}" velocity="100.0"/>
 </joint>
@@ -650,5 +650,5 @@
   <parent link="r_hipjointupper"/>
   <child link="r_hipjointlower"/>
-  <axis xyz="1.0 0.0 0.0"/>
+  <axis xyz="-1.0 0.0 0.0"/>
   <limit effort="1000" lower="${radians(-90)}" upper="${radians(90)}" velocity="100.0"/>
 </joint>
@@ -657,5 +657,5 @@
   <parent link="r_hipjointlower"/>
   <child link="r_upperreg"/>
-  <axis xyz="0.0 -1.0 0.0"/>
+  <axis xyz="0.0 1.0 0.0"/>
   <limit effort="1000" lower="${radians(-90)}" upper="${radians(90)}" velocity="100.0"/>
 </joint>
@@ -678,5 +678,5 @@
   <parent link="r_ankle"/>
   <child link="r_foot"/>
-  <axis xyz="1.0 0.0 0.0"/>
+  <axis xyz="-1.0 0.0 0.0"/>
   <limit effort="1000" lower="${radians(-90)}" upper="${radians(90)}" velocity="100.0"/>
 </joint>
